File: mcuc_inverter/gate_drive.kicad_sch (KiCad schematic)
At the start: 0 parts

Commit message: Capture gate_drive sheet: 6x 1ED3491MC12M channels, root wiring
Pinout verified from the 1ED34x1Mx12M datasheet v1.20 (single IN pin;
RDYC is dual-function ready-output / fault-clear-input, bused per
datasheet with a 1k series resistor to the supervisor's push-pull
DRV_RST_OUT). Per channel: D018 turn-on RC delay (1k/330p [TBV] with
on-sheet retune note), ON/OFF split gate resistors 12R/3R3, BSS138
Miller clamp to VEE2 per datasheet 4.5.4.1, DESAT chain (1k + 2x
US1M) to the module drain-sense pins, ADJA 4.87k (349 mA soft-off)
and ADJB 1.33k (650 ns LEB) [TBV], +18/-5 rails per HS channel with
shared LS supply. FLT_N wired-AND joins the supervisor fault
conditioning.

Root sheet: supervisor -> gate_drive (gated PWM x6, DRV_FAULT_IN,
DRV_RST_OUT) and gate_drive -> power_stage (GATE/KSRC/DSENSE x6)
wired; VGD_* rails await aux_power.

ERC 0 errors; 244/244 per-channel netlist checks by the capture
agent, key nets independently re-verified before commit.

Co-Authored-By: Claude Fable 5 <noreply@anthropic.com>
Parts:
- added C311, C321, C331, C341, C351, C361: 330p [TBV], Capacitor_SMD:C_0603_1608Metric, symbol Device:C
- added C312, C314, C316, C322, C324, C326, C332, C334, C336, C342, C344, C346, C352, C354, C356, C362, C364, C366: 100n, Capacitor_SMD:C_0603_1608Metric, symbol Device:C
- added C313, C315, C323, C325, C333, C335, C343, C345, C353, C355, C363, C365: 1u, Capacitor_SMD:C_0805_2012Metric, symbol Device:C
- added C317, C327, C337, C347, C357, C367: 100p [TBV], Capacitor_SMD:C_0603_1608Metric, symbol Device:C
- added D311, D321, D331, D341, D351, D361: BAS316, Diode_SMD:D_SOD-323, symbol Device:D
- added D312, D313, D322, D323, D332, D333, D342, D343, D352, D353, D362, D363: US1M [TBV], Diode_SMD:D_SMA, symbol Device:D
- added Q311, Q321, Q331, Q341, Q351, Q361: BSS138 [TBV], Package_TO_SOT_SMD:SOT-23, symbol Transistor_FET:BSS138
- added R311, R321, R331, R341, R351, R361: 1k [TBV], Resistor_SMD:R_0603_1608Metric, symbol Device:R
- added R312, R322, R332, R342, R352, R362: 4.87k [TBV], Resistor_SMD:R_0603_1608Metric, symbol Device:R
- added R313, R323, R333, R343, R353, R363: 1.33k [TBV], Resistor_SMD:R_0603_1608Metric, symbol Device:R
- added R314, R324, R334, R344, R354, R364: 12 [TBV], Resistor_SMD:R_1206_3216Metric, symbol Device:R
- added R315, R325, R335, R345, R355, R365: 3.3 [TBV], Resistor_SMD:R_1206_3216Metric, symbol Device:R
- added R316, R326, R336, R346, R356, R366: 1k [TBV], Resistor_SMD:R_1206_3216Metric, symbol Device:R
- added R391, R392: 4.7k, Resistor_SMD:R_0603_1608Metric, symbol Device:R
- added R393: 1k, Resistor_SMD:R_0603_1608Metric, symbol Device:R
- added U301, U302, U303, U304, U305, U306: 1ED3491MC12M, Package_SO:SOIC-16W_7.5x10.3mm_P1.27mm, symbol mcuc:1ED3491MC12M
Connections:
- new net: D342.1 (K), D343.2 (A)
- new net: D342.2 (A), R346.2
- new net: R335.1, U303.11 (OFF)
- new net: C361.1, D361.2 (A), R361.2, U306.7 (IN)
- new net: Q321.1 (G), U302.10 (CLAMPDRV)
- new net: R325.1, U302.11 (OFF)
- new net: R324.1, U302.12 (ON)
- new net: C327.1, R326.1, U302.13 (DESAT)
- new net: R322.1, U302.3 (ADJA)
- new net: R323.1, U302.4 (ADJB)
- new net: C321.1, D321.2 (A), R321.2, U302.7 (IN)
- new net: C311.1, D311.2 (A), R311.2, U301.7 (IN)
- new net: R332.1, U303.3 (ADJA)
- new net: C351.1, D351.2 (A), R351.2, U305.7 (IN)
- new net: R315.1, U301.11 (OFF)
- new net: R362.1, U306.3 (ADJA)
- new net: C331.1, D331.2 (A), R331.2, U303.7 (IN)
- new net: C367.1, R366.1, U306.13 (DESAT)
- new net: D362.2 (A), R366.2
- new net: R363.1, U306.4 (ADJB)
- new net: R343.1, U304.4 (ADJB)
- new net: D312.1 (K), D313.2 (A)
- new net: Q331.1 (G), U303.10 (CLAMPDRV)
- new net: R334.1, U303.12 (ON)
- new net: C337.1, R336.1, U303.13 (DESAT)
- new net: R333.1, U303.4 (ADJB)
- new net: R314.1, U301.12 (ON)
- new net: D332.2 (A), R336.2
- new net: R345.1, U304.11 (OFF)
- new net: R355.1, U305.11 (OFF)
- new net: Q351.1 (G), U305.10 (CLAMPDRV)
- new net: R354.1, U305.12 (ON)
- new net: C357.1, R356.1, U305.13 (DESAT)
- new net: R352.1, U305.3 (ADJA)
- new net: R353.1, U305.4 (ADJB)
- new net: D362.1 (K), D363.2 (A)
- new net: R344.1, U304.12 (ON)
- new net: C341.1, D341.2 (A), R341.2, U304.7 (IN)
- new net: D332.1 (K), D333.2 (A)
- new net: Q311.1 (G), U301.10 (CLAMPDRV)
- new net: Q361.1 (G), U306.10 (CLAMPDRV)
- new net: Q341.1 (G), U304.10 (CLAMPDRV)
- new net: R342.1, U304.3 (ADJA)
- new net: R313.1, U301.4 (ADJB)
- new net: C347.1, R346.1, U304.13 (DESAT)
- new net: D322.1 (K), D323.2 (A)
- new net: R365.1, U306.11 (OFF)
- new net: R364.1, U306.12 (ON)
- new net: D312.2 (A), R316.2
- new net: C317.1, R316.1, U301.13 (DESAT)
- new net: R312.1, U301.3 (ADJA)
- new net: D322.2 (A), R326.2
- new net: D352.1 (K), D353.2 (A)
- new net: D352.2 (A), R356.2
- new net +3.3V: C312.1, C322.1, C332.1, C342.1, C352.1, C362.1, R391.1, R392.1, U301.2 (VCC1), U302.2 (VCC1), U303.2 (VCC1), U304.2 (VCC1), U305.2 (VCC1), U306.2 (VCC1)
- new net DRV_FAULT_IN: R391.2, U301.6 (FLT_N), U302.6 (FLT_N), U303.6 (FLT_N), U304.6 (FLT_N), U305.6 (FLT_N), U306.6 (FLT_N)
- new net DRV_RST_OUT: R393.1
- new net DSENSE_HS_1: D313.1 (K)
- new net DSENSE_HS_2: D323.1 (K)
- new net DSENSE_HS_3: D333.1 (K)
- new net DSENSE_LS_1: D343.1 (K)
- new net DSENSE_LS_2: D353.1 (K)
- new net DSENSE_LS_3: D363.1 (K)
- new net GATE_HS_1: Q311.3 (D), R314.2, R315.2
- new net GATE_HS_2: Q321.3 (D), R324.2, R325.2
- new net GATE_HS_3: Q331.3 (D), R334.2, R335.2
- new net GATE_LS_1: Q341.3 (D), R344.2, R345.2
- new net GATE_LS_2: Q351.3 (D), R354.2, R355.2
- new net GATE_LS_3: Q361.3 (D), R364.2, R365.2
- new net GND: C311.2, C312.2, C321.2, C322.2, C331.2, C332.2, C341.2, C342.2, C351.2, C352.2, C361.2, C362.2, R312.2, R313.2, R322.2, R323.2, R332.2, R333.2, R342.2, R343.2, R352.2, R353.2, R362.2, R363.2, U301.1 (GND1), U301.8 (GND1), U302.1 (GND1), U302.8 (GND1), U303.1 (GND1), U303.8 (GND1), U304.1 (GND1), U304.8 (GND1), U305.1 (GND1), U305.8 (GND1), U306.1 (GND1), U306.8 (GND1)
- new net KSRC_HS_1: C313.2, C314.2, C315.1, C316.1, C317.2, U301.15 (GND2)
- new net KSRC_HS_2: C323.2, C324.2, C325.1, C326.1, C327.2, U302.15 (GND2)
- new net KSRC_HS_3: C333.2, C334.2, C335.1, C336.1, C337.2, U303.15 (GND2)
- new net KSRC_LS_1: C343.2, C344.2, C345.1, C346.1, C347.2, C353.2, C354.2, C355.1, C356.1, C357.2, C363.2, C364.2, C365.1, C366.1, C367.2, U304.15 (GND2), U305.15 (GND2), U306.15 (GND2)
- new net PWM_HS_1_GATED: D311.1 (K), R311.1
- new net PWM_HS_2_GATED: D321.1 (K), R321.1
- new net PWM_HS_3_GATED: D331.1 (K), R331.1
- new net PWM_LS_1_GATED: D341.1 (K), R341.1
- new net PWM_LS_2_GATED: D351.1 (K), R351.1
- new net PWM_LS_3_GATED: D361.1 (K), R361.1
- new net RDYC_BUS: R392.2, R393.2, U301.5 (RDYC), U302.5 (RDYC), U303.5 (RDYC), U304.5 (RDYC), U305.5 (RDYC), U306.5 (RDYC)
- new net VGD_HS1_N: C315.2, C316.2, Q311.2 (S), U301.16 (VEE2), U301.9 (VEE2)
- new net VGD_HS1_P: C313.1, C314.1, U301.14 (VCC2)
- new net VGD_HS2_N: C325.2, C326.2, Q321.2 (S), U302.16 (VEE2), U302.9 (VEE2)
- new net VGD_HS2_P: C323.1, C324.1, U302.14 (VCC2)
- new net VGD_HS3_N: C335.2, C336.2, Q331.2 (S), U303.16 (VEE2), U303.9 (VEE2)
- new net VGD_HS3_P: C333.1, C334.1, U303.14 (VCC2)
- new net VGD_LS_N: C345.2, C346.2, C355.2, C356.2, C365.2, C366.2, Q341.2 (S), Q351.2 (S), Q361.2 (S), U304.16 (VEE2), U304.9 (VEE2), U305.16 (VEE2), U305.9 (VEE2), U306.16 (VEE2), U306.9 (VEE2)
- new net VGD_LS_P: C343.1, C344.1, C353.1, C354.1, C363.1, C364.1, U304.14 (VCC2), U305.14 (VCC2), U306.14 (VCC2)
Other:
- note added: "Ch 1 - HS U (module G1 / S1.1 / D1)"
- note added: "Ch 2 - HS V (module G3 / S3.1 / D3)"
- note added: "Ch 3 - HS W (module G5 / S5.1 / D5)"
- note added: "Ch 4 - LS U (module G2 / S2.1 / D2)"
- note added: "Ch 5 - LS V (module G4 / S4.1 / D4)"
- note added: "Ch 6 - LS W (module G6 / S6.1 / D6)"
- note added: "Fault / reset aggregation (all six drivers)"
- note added: "SPEC.md 5, 9.2 - DECISIONS.md D016 / D017 / D018"
- note added: "Six isolated SiC gate-drive channels - Infineon 1ED3491MC12M (D017) driving FS02MR12A8MA2B (D016). Datasheet refs = 1ED34x1Mc12M ds v1.20. Supplies: +18 V (VGD_*_P) / -5 V (VGD_*_N) per D017, VGD_*_COM = Kelvin-source reference (= KSRC_*). HS channels: individual isolated supplies. LS channels share VGD_LS_* (Kelvin sources at common DC- potential; KSRC_LS_1/2/3 tie together on the shared COM by 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"
- note removed: "Placeholder. Requirements: SPEC.md 5"

Commit message: Board-prep: footprint audit complete, HV terminals, off-board flags
474-component audit: 466 valid resolved footprints, 13 off-board
exclusions per D024 (caps to carrier, chassis resistors, HOYS), 4
flagged TBDs (custom flyback + 3 unchosen inductors), zero silent
gaps. Netlist-fatal fixes: Q403 renumbered to Wolfspeed TO-263-7
convention (G1/KS2/S3-7/tab-D8), CSD18543Q3A remapped to KiCad's
SSSGD VSON-8 pairing - both verified in the netlist afterward.

New HV interface terminals J401-J405 (M4 ring-lug pads: DC input,
precharge-R chassis loop, discharge-R return, bus taps) and HOYS
harness headers J501-J503 (JST 2mm; PA-vs-PH footprint flagged TBV)
with net membership machine-verified incl. the OC_TRIP wire-OR and
I_REF paths to the MCU ADCs.

ERC 0 errors, warnings 201 -> 200 (none introduced).

Co-Authored-By: Claude Fable 5 <noreply@anthropic.com>
Parts:
- U301, U302, U303, U304, U305, U306: footprint Package_SO:SOIC-16W_7.5x10.3mm_P1.27mm -> mcuc:PG-DSO-16-28
Changed lines of the file:
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@@
 			)
 		)
-		(property "Footprint" "Package_SO:SOIC-16W_7.5x10.3mm_P1.27mm"
+		(property "Footprint" "mcuc:PG-DSO-16-28"
 			(at 78.74 58.42 0)
 			(effects
@@
 			)
 		)
-		(property "Footprint" "Package_SO:SOIC-16W_7.5x10.3mm_P1.27mm"
+		(property "Footprint" "mcuc:PG-DSO-16-28"
 			(at 212.09 58.42 0)
 			(effects
@@
 			)
 		)
-		(property "Footprint" "Package_SO:SOIC-16W_7.5x10.3mm_P1.27mm"
+		(property "Footprint" "mcuc:PG-DSO-16-28"
 			(at 345.44 58.42 0)
 			(effects
@@
 			)
 		)
-		(property "Footprint" "Package_SO:SOIC-16W_7.5x10.3mm_P1.27mm"
+		(property "Footprint" "mcuc:PG-DSO-16-28"
 			(at 78.74 185.42 0)
 			(effects
@@
 			)
 		)
-		(property "Footprint" "Package_SO:SOIC-16W_7.5x10.3mm_P1.27mm"
+		(property "Footprint" "mcuc:PG-DSO-16-28"
 			(at 212.09 185.42 0)
 			(effects
@@
 			)
 		)
-		(property "Footprint" "Package_SO:SOIC-16W_7.5x10.3mm_P1.27mm"
+		(property "Footprint" "mcuc:PG-DSO-16-28"
 			(at 345.44 185.42 0)
 			(effects

Commit message: Gate drive: DESAT blanking caps 100pF -> 22pF (partial CR-2 fix)
First item of the review fix pass to land before the agent was
interrupted. Reduces the DESAT ramp from 1.84 us to 272 ns.

INCOMPLETE against review 3's CR-2: with ADJB still at 1.33k
(tDESATfilter 1575 ns) and ADJA at 4.87k (349 mA soft-off), the
total detect-to-gate-off chain is still ~4.2 us against the
module's 1.2 us short-circuit withstand. Remaining work: tie ADJB
to VCC1, ADJA -> 28.0k, and either derate VGS(on) to +15 V (buys
the 2 us rating) or reopen D017 for a SiC-threshold driver
(UCC21755-Q1 at 5.0 V or STGAP3SXS at 6.0 V, both already
qualified in SPEC 5).

Also ignores KiCad's fp-info-cache.

Co-Authored-By: Claude Fable 5 <noreply@anthropic.com>
Parts:
- C317, C327, C337, C347, C357, C367: value 100p [TBV] -> 22p 50V C0G
Changed lines of the file:
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@@
 			)
 		)
-		(property "Value" "100p [TBV]"
+		(property "Value" "22p 50V C0G"
 			(at 107.95 72.898 0)
 			(effects
@@
 			)
 		)
-		(property "Value" "100p [TBV]"
+		(property "Value" "22p 50V C0G"
 			(at 241.3 72.898 0)
 			(effects
@@
 			)
 		)
-		(property "Value" "100p [TBV]"
+		(property "Value" "22p 50V C0G"
 			(at 374.65 72.898 0)
 			(effects
@@
 			)
 		)
-		(property "Value" "100p [TBV]"
+		(property "Value" "22p 50V C0G"
 			(at 107.95 199.898 0)
 			(effects
@@
 			)
 		)
-		(property "Value" "100p [TBV]"
+		(property "Value" "22p 50V C0G"
 			(at 241.3 199.898 0)
 			(effects
@@
 			)
 		)
-		(property "Value" "100p [TBV]"
+		(property "Value" "22p 50V C0G"
 			(at 374.65 199.898 0)
 			(effects

Commit message: Fix gate drive and supervisor: CR-1, CR-2, MJ-1, MJ-8, MJ-9, MJ-13
CR-1 - the fault-clear deadlock is broken. U903 gate 4 now computes
DRV_RST_OUT = DRV_RST_IN AND OC_LATCH_N; FAULT_BKIN is out of the
chain, so a rising RDYC edge is reachable. C907 (220 nF) gives a
1.03 ms power-on clear pulse, comfortably past the drivers' 200 us
start time and the 1.2 us minimum clear width, so the bridge comes
up without firmware intervention. Gate 3 is freed and labelled for
the discharge interlock.

MJ-1 - the overcurrent trip finally reaches TIM1_BKIN. D904 (BAT54WS)
wire-ORs OC_LATCH_N into FAULT_BKIN: 0.33 mA gives 0.31 V against a
0.95 V input-low threshold, and it reverse-biases on driver-only
faults so the two paths stay independent. SPEC 9.2's central claim is
now true as built.

CR-2 - DESAT reconfigured: ADJB linked to VCC1 (LEB 444 ns, filter
263 ns, was 650+1575), ADJA to 28.0k for the family-maximum 699 mA
soft-off, and the external blanking cap DNP'd because the datasheet
specifies all DESAT timing at 2 pF. Chain is now 1.9 us typical
against ~5.8 us before. Worst-case silicon reaches 2.6 us - see the
D026 amendment in the next commit; this is recorded, not rounded.

MJ-8 - added the VCC2-to-VEE2 capacitors that were missing on all six
domains. That is the loop carrying the gate pulse, and the datasheet
explicitly requires it.

MJ-9 - the -5 V off-rail had no defined bias: gate charge nets to zero
at COM, so the zener sat in its knee. 2.49k preloads (6.02 mA) per
isolated domain now hold it defined at 4.87 V, inside the module's
-5 V static maximum.

MJ-13 - LED resistors 100R -> 2.2k and D903 moved ahead of R910. The
fault wire-OR was being back-fed ~11 mA, pushing FAULT_BKIN to 0.94 V
against a 0.99 V threshold; it now sits at ~0.1 V.

MJ-17 - Miller clamp BSS138 -> BSS316N. Note the constraint the agent
found: CLAMPDRV swings to VEE2+11.5 V, so the +-12 V Vgs parts
suggested elsewhere are unusable; this is a +-20 V part.

MN-2 - documentation corrected to the tr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
Parts:
- added C318, C328, C338, C348, C358, C368: 1u 50V X7R, Capacitor_SMD:C_0805_2012Metric, symbol Device:C
- added C319, C329, C339, C349, C359, C369: 100n 50V X7R, Capacitor_SMD:C_0603_1608Metric, symbol Device:C
- added R317, R327, R337, R347: 2.49k 1% (zener preload 6.0mA), Resistor_SMD:R_1206_3216Metric, symbol Device:R
- C317, C327, C337, C347, C357, C367: value 22p 50V C0G -> 22p 50V C0G - DNP; now not fitted
- Q311, Q321, Q331, Q341, Q351, Q361: value BSS138 [TBV] -> BSS316N
- R312, R322, R332, R342, R352, R362: value 4.87k [TBV] -> 28.0k 1% (ADJA: soft-off 699mA)
- R313, R323, R333, R343, R353, R363: value 1.33k [TBV] -> 0R link (ADJB=VCC1)
- R314, R324, R334, R344, R354, R364: value 12 [TBV] -> 12R 1% 0.75W CRCW1206-HP
- R315, R325, R335, R345, R355, R365: value 3.3 [TBV] -> 3R3 1% 0.75W CRCW1206-HP
Connections:
- net +3.3V: now also R313.2, R323.2, R333.2, R343.2, R353.2, R363.2
- net GND: no longer R313.2, R323.2, R333.2, R343.2, R353.2, R363.2
- net KSRC_HS_1: now also R317.2
- net KSRC_HS_2: now also R327.2
- net KSRC_HS_3: now also R337.2
- net KSRC_LS_1: now also R347.2
- net VGD_HS1_N: now also C319.1
- net VGD_HS1_P: now also C318.2, R317.1
- net VGD_HS2_N: now also C329.1
- net VGD_HS2_P: now also C328.2, R327.1
- net VGD_HS3_N: now also C339.1
- net VGD_HS3_P: now also C338.2, R337.1
- net VGD_LS_N: now also C349.1, C359.1, C369.1
- net VGD_LS_P: now also C348.2, C358.2, C368.2, R347.1
- net RDYC_BUS renamed DRV_READY
- new net: C338.1, C339.2
- new net: C368.1, C369.2
- new net: C328.1, C329.2
- new net: C348.1, C349.2
- new net: C318.1, C319.2
- new net: C358.1, C359.2
Other:
- note added: "DRV_READY = RDYC_BUS to a free MCU GPIO (MN-18): a gate-supply UVLO pulls RDYC low without ever asserting FLT_N, so it is otherwise invisible to firmware. ROOT SHEET must add the matching sheet pin (PB10 / PB11 / PE1 are free)."
- note added: "LS domain preload is R347 (ch 4) - one per isolated rail."
- note added: "P-N decoupling (MJ-8) - the loop the gate pulse flows in."
- note added: "Six isolated SiC gate-drive channels - Infineon 1ED3491MC12M (D017) driving FS02MR12A8MA2B (D016). Datasheet refs = 1ED34x1Mc12M ds v1.20. GATE LEVELS +15 V / -5 V (was +18/-5). The module's short-circuit withstand is 1.2 us at -5/+18 V but 2 us at -5/+15 V; the DESAT chain below cannot clear inside 1.2 us at any setting of this driver, so the drive is derated to +15 V to buy the 2 us rating. Cos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"
- note added: "VGD_HS1 split-zener preload: 15 V / 2.49k = 6.0 mA, 90 mW."
- note added: "VGD_HS2 split-zener preload: 15 V / 2.49k = 6.0 mA, 90 mW."
- note added: "VGD_HS3 split-zener preload: 15 V / 2.49k = 6.0 mA, 90 mW."
- note added: "VGD_LS split-zener preload: 15 V / 2.49k = 6.0 mA, 90 mW."
- note removed: "Six isolated SiC gate-drive channels - Infineon 1ED3491MC12M (D017) driving FS02MR12A8MA2B (D016). Datasheet refs = 1ED34x1Mc12M ds v1.20. Supplies: +18 V (VGD_*_P) / -5 V (VGD_*_N) per D017, VGD_*_COM = Kelvin-source reference (= KSRC_*). HS channels: individual isolated supplies. LS channels share VGD_LS_* (Kelvin sources at common DC- potential; KSRC_LS_1/2/3 tie together on the shared COM by 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"
