File: mcuc_inverter/bus_sense.kicad_sch (KiCad schematic)
At the start: 21 parts, among them U701 AMC1311BDWV, U702 MCP1804T-3302I/OT, U703 TLV9061/OPA320-class [TBV]

Commit message: Fix aux power and bus sense per adversarial review (CR-4..7, MJ-5..22)
CR-6: real footprints for every HV part that had an impossible one -
C601/C602 (0.68 uF 630 V X2) onto the 26.5x10.5/P22.5 radial box, and
the InnoSwitch bypass caps off 0603 per the datasheet's explicit "0805
or larger, do not use 0603 rated MLCC".

CR-4: RCD clamp rebuilt as 6x 39k 1206 in 3s2p (58.5k) - worst-case
0.35 W and 117 V per part, inside a 200 V 0.5 W part everywhere,
against 0603s that were at 7.5x their voltage rating. Drain lands
731-806 V depending on leakage, so the T601 purchase spec now needs
L_k <= 2 uH; recorded on-sheet.

CR-5 solved better than directed: the agent found the -AQ family has
no reduced current-limit setting, so swapping to INN3999CQ was the
wrong premise. Changing the BPP capacitor 4.7 -> 0.47 uF selects the
standard limit, giving B_pk 360 mT typ (below DER-948Q's own 376 mT
design point) while keeping MORE power headroom than the part swap
would have. Controller retained.

CR-7: both bucks LMR51430 SOT-23-6 -> LMR33630ADDAR HSOIC-8 PowerPAD
(42.9 vs 107.8 C/W), new verified symbol, thermal pad wired as AGND
per Table 6-1. Dividers, 10 uH inductors and 10 uF + 220 nF input
capacitance per Table 9-2.

MJ-14: flyback line UV/OV sensing enabled (the V pin was tied to
SOURCE, which the reference design warns makes regulation fail below
80 V while SPEC requires 48 V). Brown-in 32.5-44.2 V over temp.

MJ-10: LM5175 current limit 10 -> 30 mOhm; it was tripping at 17 A
against a 7.6 A inductor saturation, so the inductor saturated before
the limit acted. MJ-5: bus-sense filter 100 nF -> 100 pF, moving the
OVP response from ~1.3 ms to ~13 us. MJ-16: C702's unconnected pin
wired - it was the LDO output capacitor whose net was never drawn.

MJ-22 deviates from my instruction, correctly: at the gain I specified
the 490 V OVP would have landed 6 mV above a -4% supply rail, i.e.
unreachable by an RRIO output. Gain 1.50 instead - 500 V -> 2.988 V,
90.5% of range, 168 mV hea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
Parts:
- C703: value 100nF -> 100pF
- R701, R702, R703, R704, R706: Tolerance (none) -> 1%
- R705, R707, R708: Tolerance (none) -> 0.1%
- R709, R710: value 7.50k -> 15.0k; Tolerance (none) -> 0.1%
Connections:
- net 3V3_HV: now also C702.1
Other:
- note added: "*** CR-3 OPEN - HV-SIDE 3.3 V SUPPLY IS STILL WRONG AS DRAWN *** U702 takes VIN from VGD_LS_P and GND from VGD_LS_COM (the module low-side Kelvin source pins) while C701/C702, the AMC1311 GND1 and the divider bottom R705 all sit on DC_BUS_N. Those nets join only through the module internals, so tens of volts appear across that loop on every switching edge, and a Kelvin sense node is being used as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"
- note added: "ACCURACY (MJ-6 / MN-19): Tolerance fields are now explicit on every resistor - 0.1% on R705 and R707-R710 (they set the ratio), 1% on the 750k string and R706. OPEN, NOT FIXABLE ON THIS SHEET: the SPEC 8.2 +/-1% figure is also gated by the ADC reference. VREF+ is the TLV1117-33 rail at +/-4%, which alone is 4x the budget. Fit a REF3033 (or equivalent) on VREF+, or calibrate the gain in firmware. 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"
- note added: "Diff-to-SE: Vout = (R709/R707) x (OUTP-OUTN) = 1.50 x VIN. R707=R708=10.0k, R709=R710=15.0k, all 0.1% E96 (CMRR is set by the ratio match). WHY NOT 16.2k (gain 1.62): 490 V would sit at 3.162 V, and a TLV1117 3.3 V rail at its -4% limit is 3.168 V - an RRIO output cannot reproduce that, so the OVP threshold would be unreachable. At gain 1.50 the maximum output is 3.000 V, i.e. 168 mV of headroom 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"
- note added: "MJ-5 FIXED: C703 100 nF -> 100 pF (TI Fig. 9-2 value). Source impedance = R706 1.0k + (12.0k || 3000k) = 12.95k. 100 nF -> tau 1.30 ms, fc 123 Hz : the 490 V OVP arrived ~1-3 ms late (363 V of lag at the 140 A regen dV/dt). 100 pF -> tau 1.30 us, fc 123 kHz, inside the AMC1311B >=220 kHz bandwidth. DO NOT fit clamp/protection diodes on IN: AMC1311 datasheet 9.3 (diode leakage corrupts the reading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"
- note added: "SCALING (MJ-22 fixed): V_BUS = Vbus x (12.0k/3012k) x 1.50 = 5.976 mV/V. 500 V -> 2.988 V | 490 V (OV trip, SPEC 9.1) -> 2.928 V | 250 V -> 1.494 V. AMC1311 input clips at 2.00 V = 502 V bus -> V_BUS saturates at 3.000 V. 12-bit ADC on a 3.3 V reference: 805.7 uV/LSB = 0.135 V of bus per LSB. Was 0.75x (500 V -> 1.494 V), which wasted 55% of the ADC range."
- note removed: "Diff-to-SE: Vout = (7.50k/10.0k) x (OUTP-OUTN) = 0.75 x VIN (OUTP/OUTN swing +/-1 V about VCM 1.44 V; common mode rejected by the 4-resistor stage, output referenced to GND). E96 0.1% for R707-R710 (CMRR set by ratio match). Op amp: any RRIO 3.3 V single in SOT-23-5 (TLV9061IDBVR primary / OPA320 [TBV])."
- note removed: "HV-side 3.3 V: MCP1804T-3302I/OT (2-28 V in, 150 mA, verified stocked 2026-08-02) from the +18 V low-side gate rail VGD_LS_P, referenced to VGD_LS_COM [TBV - noise review, D022]. AMC1311 GND1 ties to DC_BUS_N (divider bottom). VGD_LS_COM and DC_BUS_N join only at the module low-side source Kelvin / N-terminal copper - supply return path is through that joint. Kelvin split + LDO PSRR review [TBV]."
- note removed: "R706/C703: input RC ahead of IN (fc ~ 120 Hz with the 12.0k tap; TI Fig. 9-2 fits only 100 pF - value TBV vs required sense bandwidth). DO NOT fit clamp/protection diodes on IN: AMC1311 datasheet 9.3 (diode leakage corrupts the reading; ESD cells + divider impedance are the specified protection)."
- note removed: "SCALING: V_BUS = Vbus x (12.0k/3012k) x 0.75 = 2.988 mV/V. 500 V -> 1.494 V | 250 V -> 0.747 V | 490 V (OV trip, SPEC 9.1) -> 1.464 V. AMC1311 input clips at 2.00 V = 502 V bus, so V_BUS saturates at ~1.50 V: always < 3.3 V ADC full scale by design (headroom deliberate, not an error)."
Changed lines of the file:
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@@
-		)
-	)
-	(text "SCALING: V_BUS = Vbus x (12.0k/3012k) x 0.75 = 2.988 mV/V.\n500 V -> 1.494 V | 250 V -> 0.747 V | 490 V (OV trip, SPEC 9.1) -> 1.464 V.\nAMC1311 input clips at 2.00 V = 502 V bus, so V_BUS saturates at ~1.50 V:\nalways < 3.3 V ADC full scale by design (headroom deliberate, not an error)."
-		(exclude_from_sim no)
-		(at 20 39.37 0)
-		(effects
-			(font
-				(size 1.27 1.27)
-			)
-			(justify left bottom)
 		)
 	)
@@
 			)
 		)
+		(property "Tolerance" "1%"
+				(at 45.72 63.5 0)
+				(effects
+					(font
+						(size 1.27 1.27)
+					)
+					(justify left)
+					(hide yes)
+				)
+		)
 		(instances
 			(project "mcuc_inverter"
@@
 			)
 		)
+		(property "Tolerance" "1%"
+				(at 45.72 73.66 0)
+				(effects
+					(font
+						(size 1.27 1.27)
+					)
+					(justify left)
+					(hide yes)
+				)
+		)
 		(instances
 			(project "mcuc_inverter"
@@
 			)
 		)
+		(property "Tolerance" "1%"
+				(at 45.72 83.82 0)
+				(effects
+					(font
+						(size 1.27 1.27)
+					)
+					(justify left)
+					(hide yes)
+				)
+		)
 		(instances
 			(project "mcuc_inverter"
@@
 				(hide yes)
 			)
+		)
+		(property "Tolerance" "1%"
+				(at 45.72 93.98 0)
+				(effects
+					(font
+						(size 1.27 1.27)
+					)
+					(justify left)
+					(hide yes)
+				)
 		)
 		(instances
@@
 				(hide yes)
 			)
+		)
+		(property "Tolerance" "0.1%"
+				(at 45.72 106.68 0)
+				(effects
+					(font
+						(size 1.27 1.27)
+					)
+					(justify left)
+					(hide yes)
+				)
 		)
 		(instances
@@
 			)
 		)
+		(property "Tolerance" "1%"
+				(at 55.88 100.33 0)
+				(effects
+					(font
+						(size 1.27 1.27)
+					)
+					(justify left)
+					(hide yes)
+				)
+		)
 		(instances
 			(project "mcuc_inverter"
@@
 			)
 		)
-		(property "Value" "100nF"
+		(property "Value" "100pF"
 			(at 66.04 105.41 0)
 			(effects
@@
 			(width 0)
 			(type default)
-		)
-	)
-	(text "R706/C703: input RC ahead of IN (fc ~ 120 Hz with the 12.0k tap;\nTI Fig. 9-2 fits only 100 pF - value TBV vs required sense bandwidth).\nDO NOT fit clamp/protection diodes on IN: AMC1311 datasheet 9.3\n(diode leakage corrupts the reading; ESD cells + divider impedance\nare the specified protection)."
-		(exclude_from_sim no)
-		(at 55.88 133.35 0)
-		(effects
-			(font
-				(size 1.0 1.0)
-			)
-			(justify left bottom)
 		)
 	)
@@
 		)
 	)
-	(text "HV-side 3.3 V: MCP1804T-3302I/OT (2-28 V in, 150 mA, verified stocked 2026-08-02)\nfrom the +18 V low-side gate rail VGD_LS_P, referenced to VGD_LS_COM [TBV - noise\nreview, D022]. AMC1311 GND1 ties to DC_BUS_N (divider bottom). VGD_LS_COM and\nDC_BUS_N join only at the module low-side source Kelvin / N-terminal copper -\nsupply return path is through that joint. Kelvin split + LDO PSRR review [TBV]."
-		(exclude_from_sim no)
-		(at 130.81 74.93 0)
-		(effects
-			(font
-				(size 1.0 1.0)
-			)
-			(justify left bottom)
-		)
-	)
 	(wire
 		(pts
@@
 				(hide yes)
 			)
+		)
+		(property "Tolerance" "0.1%"
+				(at 137.16 100.33 0)
+				(effects
+					(font
+						(size 1.27 1.27)
+					)
+					(justify left)
+					(hide yes)
+				)
 		)
 		(instances
@@
 			)
 		)
-		(property "Value" "7.50k"
+		(property "Value" "15.0k"
 			(at 143.51000000000002 113.03 0)
 			(effects
@@
 			)
 		)
+		(property "Tolerance" "0.1%"
+				(at 146.05 111.76 0)
+				(effects
+					(font
+						(size 1.27 1.27)
+					)
+					(justify left)
+					(hide yes)
+				)
+		)
 		(instances
 			(project "mcuc_inverter"
@@
 				(hide yes)
 			)
+		)
+		(property "Tolerance" "0.1%"
+				(at 137.16 105.41 0)
+				(effects
+					(font
+						(size 1.27 1.27)
+					)
+					(justify left)
+					(hide yes)
+				)
 		)
 		(instances
@@
 			)
 		)
-		(property "Value" "7.50k"
+		(property "Value" "15.0k"
 			(at 163.83 86.868 270)
 			(effects
@@
 				(hide yes)
 			)
+		)
+		(property "Tolerance" "0.1%"
+				(at 160.02 90.17 0)
+				(effects
+					(font
+						(size 1.27 1.27)
+					)
+					(justify left)
+					(hide yes)
+				)
 		)
 		(instances
@@
 		)
 	)
-	(text "Diff-to-SE: Vout = (7.50k/10.0k) x (OUTP-OUTN) = 0.75 x VIN (OUTP/OUTN swing +/-1 V about VCM 1.44 V; common mode rejected by the 4-resistor stage,\noutput referenced to GND). E96 0.1% for R707-R710 (CMRR set by ratio match). Op amp: any RRIO 3.3 V single in SOT-23-5 (TLV9061IDBVR primary / OPA320 [TBV])."
-		(exclude_from_sim no)
-		(at 130.81 127.0 0)
+	(text "AMC1311 failsafe: OUTP-OUTN = -2.5 V (V_BUS pulled to 0 V) when the high side is unpowered\nor SHTDN asserted - firmware reads a dead bus, which is the safe direction for the 45 V UV inhibit."
+		(exclude_from_sim no)
+		(at 130.81 133.35 0)
 		(effects
 			(font
@@
 		)
 	)
-	(text "AMC1311 failsafe: OUTP-OUTN = -2.5 V (V_BUS pulled to 0 V) when the high side is unpowered\nor SHTDN asserted - firmware reads a dead bus, which is the safe direction for the 45 V UV inhibit."
-		(exclude_from_sim no)
-		(at 130.81 133.35 0)
+	(wire
+		(pts
+			(xy 111.76 60.96) (xy 111.76 58.42)
+		)
+		(stroke
+			(width 0)
+			(type default)
+		)
+	)
+	(text "SCALING (MJ-22 fixed): V_BUS = Vbus x (12.0k/3012k) x 1.50 = 5.976 mV/V.\n500 V -> 2.988 V | 490 V (OV trip, SPEC 9.1) -> 2.928 V | 250 V -> 1.494 V.\nAMC1311 input clips at 2.00 V = 502 V bus -> V_BUS saturates at 3.000 V.\n12-bit ADC on a 3.3 V reference: 805.7 uV/LSB = 0.135 V of bus per LSB.\nWas 0.75x (500 V -> 1.494 V), which wasted 55% of the ADC range."
+		(exclude_from_sim no)
+		(at 20 39.37 0)
 		(effects
 			(font
+				(size 1.27 1.27)
+			)
+			(justify left bottom)
+		)
+	)
+	(text "MJ-5 FIXED: C703 100 nF -> 100 pF (TI Fig. 9-2 value).\nSource impedance = R706 1.0k + (12.0k || 3000k) = 12.95k.\n  100 nF -> tau 1.30 ms, fc 123 Hz : the 490 V OVP arrived ~1-3 ms late\n            (363 V of lag at the 140 A regen dV/dt).\n  100 pF -> tau 1.30 us, fc 123 kHz, inside the AMC1311B >=220 kHz bandwidth.\nDO NOT fit clamp/protection diodes on IN: AMC1311 datasheet 9.3 (diode leakage\ncorrupts the reading; ESD cells + divider impedance are the specified protection)."
+		(exclude_from_sim no)
+		(at 55.88 133.35 0)
+		(effects
+			(font
+				(size 1.0 1.0)
+			)
+			(justify left bottom)
+		)
+	)
+	(text "Diff-to-SE: Vout = (R709/R707) x (OUTP-OUTN) = 1.50 x VIN.  R707=R708=10.0k,\nR709=R710=15.0k, all 0.1% E96 (CMRR is set by the ratio match).\nWHY NOT 16.2k (gain 1.62): 490 V would sit at 3.162 V, and a TLV1117 3.3 V rail at\nits -4% limit is 3.168 V - an RRIO output cannot reproduce that, so the OVP\nthreshold would be unreachable.  At gain 1.50 the maximum output is 3.000 V, i.e.\n168 mV of headroom even on the worst-case rail, and 90.5% of the ADC span is used.\nOp amp: RRIO 3.3 V single in SOT-23-5 (TLV9061IDBVR primary / OPA320 [TBV]);\nload is 200 uA, so the output swings to within ~20 mV of the rails."
+		(exclude_from_sim no)
+		(at 130.81 127 0)
+		(effects
+			(font
+				(size 1.0 1.0)
+			)
+			(justify left bottom)
+		)
+	)
+	(text "ACCURACY (MJ-6 / MN-19): Tolerance fields are now explicit on every resistor -\n0.1% on R705 and R707-R710 (they set the ratio), 1% on the 750k string and R706.\nOPEN, NOT FIXABLE ON THIS SHEET: the SPEC 8.2 +/-1% figure is also gated by the ADC\nreference.  VREF+ is the TLV1117-33 rail at +/-4%, which alone is 4x the budget.\nFit a REF3033 (or equivalent) on VREF+, or calibrate the gain in firmware.\nThis is an MCU-sheet / SPEC change and is reported, not implemented here."
+		(exclude_from_sim no)
+		(at 20 152.4 0)
+		(effects
+			(font
+				(size 1.0 1.0)
+			)
+			(justify left bottom)
+		)
+	)
+	(text "*** CR-3 OPEN - HV-SIDE 3.3 V SUPPLY IS STILL WRONG AS DRAWN ***\nU702 takes VIN from VGD_LS_P and GND from VGD_LS_COM (the module low-side Kelvin\nsource pins) while C701/C702, the AMC1311 GND1 and the divider bottom R705 all sit\non DC_BUS_N.  Those nets join only through the module internals, so tens of volts\nappear across that loop on every switching edge, and a Kelvin sense node is being\nused as a power node.  Moving only U702 GND to DC_BUS_N does not fix it - the same\ntransient then appears across VIN-GND.\nREQUIRED (TI SBAS786C 10, and D022 already flags this [TBV]):\n  - a fifth SN6505B push-pull stage whose SECONDARY is referenced to DC_BUS_N,\n    primary from the control-side +5V/GND (load is only <=8.4 mA);\n  - transformer Wurth 750313734: 1:1.1, 340 uH, 5000 Vrms hipot, REINFORCED\n    800 Vrms per IEC62368-1, 9.2 mm creepage / 8.0 mm clearance per IEC61800-5-1.\n    A 2.5 kV-class part (e.g. 760390012) is only FUNCTIONAL insulation and must\n    not be used: this transformer physically bridges the SPEC 10 reinforced\n    barrier at 450 V working.\n  - Schottky full-wave rectifier -> ~5.5 V raw, then U702 (MCP1804T-3302I/OT,\n    already verified stocked) to 3V3_HV, referenced to DC_BUS_N throughout;\n  - delete the VGD_LS_P and VGD_LS_COM hierarchical labels from this sheet.\nNOT IMPLEMENTED: the Wurth 750313734 land pattern could not be verified against the\nmanufacturer drawing in this pass, and a guessed footprint for a reinforced-barrier\npart is not acceptable.  C702 pin 1 (MJ-16) has been wired to the LDO output, which\nis correct in either topology."
+		(exclude_from_sim no)
+		(at 130.81 74.93 0)
+		(effects
+			(font

Commit message: CR-3: dedicated isolated supply for the bus-sense amplifier
The AMC1311's high-side LDO had VIN on VGD_LS_P and GND on
VGD_LS_COM - the module's low-side Kelvin-source pins - while its own
output capacitors, the amplifier's GND1 and the divider bottom all
sat on DC_BUS_N. Those are different nets joined only through the
module's internal copper, so at 4 kA/us across ~8 nH of source
inductance tens of volts appeared inside the supply loop every
switching edge, and a Kelvin sense node was carrying power current.

Replaced with the pattern TI actually recommends: an SN6505B
push-pull stage from the LV 5 V rail through a Wuerth 750313734
transformer, rectified and post-regulated to 3.3 V, with everything
on the isolated side referenced to DC_BUS_N. Netlist confirms one
node carrying the LDO ground, all four bypass capacitors, the
divider bottom, the amplifier's GND1 and the transformer's secondary
centre tap.

The transformer is the barrier-crossing element, so it is a genuinely
reinforced part - 800 Vrms/1400 Vpk per IEC62368-1, 5000 Vrms hipot,
9.2 mm creepage - not one of the 2.5 kV-class parts whose hipot
number masks functional-only certification. Its footprint was built
from pad coordinates rendered off the manufacturer drawing and
re-read numerically from the generated file rather than eyeballed.

Root sheet: the now-obsolete VGD_LS_P and VGD_LS_COM pins removed
from the bus_sense sheet symbol. ERC 0 errors.

Sourcing note for the BOM: SN6505BDBVR is on DigiKey backorder at
check; LCSC stocks it.

Co-Authored-By: Claude Fable 5 <noreply@anthropic.com>
Parts:
- added C711, C713: 10uF, Capacitor_SMD:C_0805_2012Metric, symbol Device:C
- added C712: 100nF, Capacitor_SMD:C_0603_1608Metric, symbol Device:C
- added D701, D702: SS310 [TBV], Diode_SMD:D_SMC, symbol Device:D_Schottky
- added T701: 750313734, mcuc:WE_750313734, symbol mcuc:WE_750313734
- added U704: SN6505BDBVR, Package_TO_SOT_SMD:SOT-23-6, symbol Power_Management:SN6505BDBV
Connections:
- net VGD_LS_COM is gone; now on net DC_BUS_N: C701.2, C702.2, U702.2 (GND)
- net DC_BUS_N: now also C713.2, T701.5 (CT_SEC)
- net GND: now also C711.2, C712.2, U704.4 (GND), U704.6 (CLK)
- net VGD_LS_P renamed 5V5_HV_RAW
- net 5V5_HV_RAW: now also C713.1, D701.1 (K), D702.1 (K)
- new net: D702.2 (A), T701.4 (SEC.E)
- new net: T701.1 (PRI.S), U704.1 (D1)
- new net: T701.3 (PRI.E), U704.3 (D2)
- new net: D701.2 (A), T701.6 (SEC.S)
- new net +5V: C711.1, C712.1, T701.2 (CT_PRI), U704.2 (VCC), U704.5 (EN)
Other:
- note added: "CR-3 - ISOLATED HIGH-SIDE SUPPLY FOR THE AMC1311 (TI SBAS786C section 10). WHY THIS STAGE EXISTS: U702 previously drew VIN/GND from VGD_LS_P / VGD_LS_COM, which are the power module LOW-SIDE KELVIN SOURCE pins. A Kelvin sense node must never carry supply current: at 4 kA/us through ~8 nH of module source inductance the Kelvin pair and DC_BUS_N differ by tens of volts on every edge, and that trans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"
- note added: "CR-3 FIXED - ISOLATED HIGH-SIDE 3.3 V SUPPLY (see stage at bottom of sheet). U702 was previously fed VIN from VGD_LS_P and GND from VGD_LS_COM, the power module low-side KELVIN SOURCE pins, while C701/C702, U701 GND1 and the divider bottom R705 sat on DC_BUS_N. Those are different nets, joined only through the module internal copper: at 4 kA/us across ~8 nH of module source inductance, tens of vo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"
- note removed: "*** CR-3 OPEN - HV-SIDE 3.3 V SUPPLY IS STILL WRONG AS DRAWN *** U702 takes VIN from VGD_LS_P and GND from VGD_LS_COM (the module low-side Kelvin source pins) while C701/C702, the AMC1311 GND1 and the divider bottom R705 all sit on DC_BUS_N. Those nets join only through the module internals, so tens of volts appear across that loop on every switching edge, and a Kelvin sense node is being used as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"
