File: mcuc_inverter/precharge.kicad_sch (KiCad schematic)
At the start: 24 parts, among them K401 HV DC precharge relay, >=450 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, Q401 AO3400-class [TBV], Q402 AO3400-class [TBV], Q403 C3M0350120J [TBV], U401 VOM1271T

Commit message: Actually apply R426 10k -> 10M (previous commit's edit had failed)
The prior commit claimed the R426 fix but the text substitution had
silently failed on a line-ending mismatch while the commit chain
proceeded. This commit contains the real change, verified in-file:
R426 (discharge FET gate pulldown) is now 10M so the VOM1271's
15-47 uA photovoltaic output can develop full gate voltage; 10k
would have held Vgs at ~0.2 V and discharge would never fire.

ERC 0 errors re-verified.

Co-Authored-By: Claude Fable 5 <noreply@anthropic.com>
Parts:
- R426: value 10k [TBV] -> 10M
Changed lines of the file:
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@@
 			)
 		)
-		(property "Value" "10k [TBV]"
+		(property "Value" "10M"
 			(at 165.1 92.71 0)
 			(effects

Commit message: Board-prep: footprint audit complete, HV terminals, off-board flags
474-component audit: 466 valid resolved footprints, 13 off-board
exclusions per D024 (caps to carrier, chassis resistors, HOYS), 4
flagged TBDs (custom flyback + 3 unchosen inductors), zero silent
gaps. Netlist-fatal fixes: Q403 renumbered to Wolfspeed TO-263-7
convention (G1/KS2/S3-7/tab-D8), CSD18543Q3A remapped to KiCad's
SSSGD VSON-8 pairing - both verified in the netlist afterward.

New HV interface terminals J401-J405 (M4 ring-lug pads: DC input,
precharge-R chassis loop, discharge-R return, bus taps) and HOYS
harness headers J501-J503 (JST 2mm; PA-vs-PH footprint flagged TBV)
with net membership machine-verified incl. the OC_TRIP wire-OR and
I_REF paths to the MCU ADCs.

ERC 0 errors, warnings 201 -> 200 (none introduced).

Co-Authored-By: Claude Fable 5 <noreply@anthropic.com>
Parts:
- added J401: DC_INPUT_P tap - 6.3mm FASTON / M4 ring lug [TBV], MountingHole:MountingHole_4.3mm_M4_Pad_Via, symbol Connector:Screw_Terminal_01x01
- added J402: to R401 chassis - 6.3mm FASTON / M4 ring lug [TBV], MountingHole:MountingHole_4.3mm_M4_Pad_Via, symbol Connector:Screw_Terminal_01x01
- added J403: R401 return to DC_BUS_P tap - 6.3mm FASTON / M4 r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, MountingHole:MountingHole_4.3mm_M4_Pad_Via, symbol Connector:Screw_Terminal_01x01
- added J404: from R424 chassis - 6.3mm FASTON / M4 ring lug [T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, MountingHole:MountingHole_4.3mm_M4_Pad_Via, symbol Connector:Screw_Terminal_01x01
- added J405: DC_BUS_N tap - 6.3mm FASTON / M4 ring lug [TBV], MountingHole:MountingHole_4.3mm_M4_Pad_Via, symbol Connector:Screw_Terminal_01x01
- K401: footprint (none) -> mcuc:HFE80V_HTPAJ
- Q403: footprint (none) -> Package_TO_SOT_SMD:TO-263-7_TabPin8
- R411, R412, R413, R414: footprint (none) -> Resistor_SMD:R_2512_6332Metric
Connections:
- net DC_BUS_N: now also Q403.3 (S), Q403.4 (S), Q403.5 (S), Q403.6 (S), Q403.7 (S), J405.1 (Pin_1)
- net DC_BUS_P: now also J403.1 (Pin_1)
- net DC_INPUT_P: now also J401.1 (Pin_1)
- net DISCHG_R_RET: now reaches R424.2
- net DISCHG_R_RET: now also Q403.8 (D), J404.1 (Pin_1); no longer Q403.3 (D)
- net PRECHG_R_CHASSIS: now reaches K401.1, R401.1
- net PRECHG_R_CHASSIS: now also J402.1 (Pin_1)
Other:
- note added: "Off-board HV interfaces (D021/D024). J401 DC input tap; J402/J403 chassis precharge resistor loop (R401 excluded from board); J404 return of chassis discharge bank R421-R424 (excluded from board) into Q403 drain; J405 DC_BUS_N tap. Bleeder R411-R414, divider and flyback taps stay on-board on the DC_BUS_P / DC_BUS_N nets behind J403/J405. Terminal footprint: M4 ring-lug pad (Pad_Via); final 6.3 mm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"

Commit message: Fix precharge, current sense, position, comms per review
Also repairs a library-breaking defect the agent found while working:
the VOM1271T symbol contained a raw newline inside a quoted string,
which silently truncated mcuc_inverter.kicad_sym at parse - every
symbol defined after it was unresolvable. That had been latent since
the symbol was written.

MJ-2/3 - the comparators were wrong twice over: TLV7032 is push-pull
(six of them wire-ORed together plus three open-drain transducer OCD
pins is direct contention), and LM2903's input common-mode range on
3.3 V stops at 1.8 V, below the 2.34 V upper threshold, so the
over-current half could never trip. Now TLV7022DDFR: true open-drain,
rail-to-rail input, 260 ns instead of ~3 us.

MJ-4 - the trip point was really 245-356 A because the thresholds
rode a +-4% rail while the transducer's reference is absolute. Each
phase's window is now servo'd off its own Uref through an OPA376
buffer, so the threshold tracks the sensor: 300 A +-8 A.

MJ-7 - a harness disconnect was not fail-safe: that phase's OCD left
the wire-OR and the input floated. 100k pull-downs make an open
harness read as a large negative current and latch the trip at
power-up, before HV is applied.

MJ-12 - the active discharge can no longer be commanded into a live
bus: SN74LVC1G97 computes DISCHARGE_EN AND NOT(CONTACTOR_EN)
self-contained on the sheet, plus a 10k boot pull-down.

Discharge gate now has a real Miller clamp (BSS138 + 1n + 10k) firing
at V_GS ~1.34 V, below the FET's 1.8 V threshold, in under 15 ns -
the 450 V dv/dt step could previously inject ~4.4 V against a 10M
pull-down and a uA-class photovoltaic turn-off.

Bleeder 18.7k -> 14k (56 k total, 56.4 s to 60 V, meeting the <60 s
requirement it was failing at 75.4 s). Precharge resistor respec'd to
>=65 J. Coil freewheels upsized to ES1G/ES2G with anti-series SMBJ24A
TVS for fast relay release, which forced the coil drivers to 60 V
parts - documented with a 17% margin note.

Position: SinCos f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
Parts:
- added C420: 100nF, Capacitor_SMD:C_0603_1608Metric, symbol Device:C
- added C421: 1nF, Capacitor_SMD:C_0603_1608Metric, symbol Device:C
- added D404, D405: SMBJ24A, Diode_SMD:D_SMB, symbol Device:D_Zener
- added Q404: BSS138, Package_TO_SOT_SMD:SOT-23, symbol mcuc:BSS138
- added R428, R429: 10k, Resistor_SMD:R_0603_1608Metric, symbol Device:R
- added U402: SN74LVC1G97DBVR, Package_TO_SOT_SMD:SOT-23-6, symbol mcuc:SN74LVC1G97DBVR
- D401: value BAS316 [TBV] -> ES1G; footprint Diode_SMD:D_SOD-323 -> Diode_SMD:D_SMA
- D402: value BAS316 [TBV] -> ES2G; footprint Diode_SMD:D_SOD-323 -> Diode_SMD:D_SMB
- D403: value MM3Z18VT1G -> MMSZ5245BT1G; footprint Diode_SMD:D_SOD-323 -> Diode_SMD:D_SOD-123
- K401: value HV DC precharge relay, >=450 V DC contacts [TBV] -> HFE80V-20C/450-12-HTPAJ
- Q401: value AO3400-class [TBV] -> NVR5198NLT1G; symbol Transistor_FET:AO3400A -> mcuc:NVR5198NL
- Q402: value AO3400-class [TBV] -> DMN6068LK3-13; footprint Package_TO_SOT_SMD:SOT-23 -> Package_TO_SOT_SMD:TO-252-3_TabPin2; symbol Transistor_FET:AO3400A -> mcuc:DMN6068LK3
- R401: value 1.25k 50W >=41J pulse [TBV] -> 1.2k 50W chassis, >=65J single-shot
- R411, R412, R413, R414: value 18.7k 3W [TBV] -> 14k 2W
- R427: value 100R -> 220R
Connections:
- net +12V: now also D404.2 (A), D405.2 (A); no longer D401.1 (K), D402.1 (K)
- net +3.3V: now also C420.1, U402.5 (VCC)
- net CONTACTOR_EN: now also U402.6 (IN2)
- net DC_BUS_N: now also Q404.2 (S), R428.2
- net DISCHARGE_EN: now also R429.1, U402.1 (IN1); no longer R427.1
- net GND: now also C420.2, R429.2, U402.2 (GND), U402.3 (IN0)
- net Q403_G: now reaches D403.1 (K), Q403.1 (G), R425.2, R426.1
- net Q403_G: now also C421.1, Q404.3 (D)
- new net: C421.2, Q404.1 (G), R428.1
- new net: D402.1 (K), D405.1 (K)
- new net: D401.1 (K), D404.1 (K)
- new net DISCHARGE_DRV: R427.1, U402.4 (Y)
Other:
- note added: "Active discharge (SPEC 7.2): R421-R424, 4 x 220R = 880R, in series with Q403 (C3M0350120J, 1200 V SiC). ~0.51 A initial at 450 V, ~230 W initial pulse for < 5 s - single-shot thermal rating [TBV], not continuous. Series string per SPEC 8.2 - no single resistor spans 450 V. HARDWARE-INHIBITED (SPEC 7.2 / D025 / review 3 MJ-12): see the DISCHARGE_DRV interlock below. Asserting DISCHARGE_EN while CO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"
- note added: "COIL DRIVER RE-RATING - consequence of the diode+TVS clamp above, NOT an independent change. Q401/Q402 were AO3400A, V_DS 30 V. With a SMBJ24A clamping at V_BR 26.7-29.5 V (and up to ~32 V at 2.5 A) plus the series rectifier V_F, the drain of each low-side switch now rests at rail + ~30-32 V during coil release: ~44 V at a nominal 12 V rail, ~48-50 V worst case on a 16 V rail. The 30 V parts woul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"
- note added: "COIL SUPPRESSION - review 3 C4/MN-5 and D025 (contactor coil is 1.7-2.5 A, SPEC 11.2, a requirement not an assumption). D401/D402 were BAS316: 250 mA I_F(AV), 500 mA I_FRM. D402 saw the full 1.7-2.5 A coil current on the first contactor drop-out - it fails, and takes Q402 with it. D401 sat at exactly its 250 mA rating. D401 -> ES1G (SMA / DO-214AC, 400 V, 1.0 A I_F(AV), 30 A I_FSM 8.3 ms, t_rr 35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"
- note added: "DISCHARGE INTERLOCK - SPEC 7.2 / D025 / review 3 MJ-12 (was CRITICAL C2). DISCHARGE_EN (PE4) and CONTACTOR_EN (PE3) were independent GPIOs with nothing between them. U402 = TI SN74LVC1G97DBVR configurable gate, SOT-23-6, 1.65-5.5 V, tpd 6.3 ns max at 3.3 V, +/-24 mA, Schmitt inputs, Ioff. Its function is Y = /IN2 . IN1 + IN2 . IN0 (a 2:1 mux, IN2 = select). TYING IN0 (pin 3) TO GND gives Y = IN1 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"
- note added: "K401 = Hongfa HFE80V-20C/450-12-HTPAJ (orderable ordering code; the Value field previously held a description). Coil is in the LV 12 V domain, contacts switch the HV DC bus - the relay itself is the isolation barrier and must be rated for it: HV DC precharge relay, >= 450 V DC contact rating, 20 A. K401 never breaks load (verified review 2). Coil suppression: D401 + D404, see the coil-suppression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"
- note added: "Passive bleeder: series string, >= 4 resistors per SPEC 8.2 - no single part may span 450 V. CORRECTED (D025 / review 3 MJ-11): 4 x 18.7k = 74.8k gave tau = 37.4 s and 75.4 s from 450 V to 60 V - it FAILED SPEC 7.2's own < 60 s requirement by 26 %. Now 4 x 14k = 56k: tau = 56k x 500 uF = 28.0 s, t(450 -> 60 V) = 28.0 x ln(450/60) = 56.4 s. 3.6 W total at 450 V; 0.90 W and 112.5 V per part. Part: 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"
- note added: "Q403 gate drive - VOM1271 photovoltaic driver, no supply needed. Rds elevated at ~8 V VGS (not spec'd below 11 V) - acceptable for current-limited single-shot duty (D022 research). R427 100R -> 220R (review 2 MJ-5 / MN-4): at 100R the LED drew I_F = 17-21 mA from an STM32F405 pin whose characterisation point is 8 mA and whose absolute maximum is 25 mA, leaving V_OC / I_SC indeterminate. The LED i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"
- note added: "R401 precharge resistor - CORRECTED (D025 / SPEC 7.1). This note previously assumed a 400 uF bank; it is 500 uF. E = 0.5 x C x V^2 = 0.5 x 500u x 450^2 = 50.6 J (53.2 J at C +5 %), and 62.5 J when precharging from a 500 V rail -> requirement is >= 65 J single-shot, NOT the >= 41 J previously printed here. Part: Ohmite/ARCOL HS50 1K2 J - 1.2k +/-5 % wirewound, aluminium housed, chassis mount, 1250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"
- note added: "SPEC 7.2 discharge requirements: Passive bleeder: < 60 V within 60 s | 56k (4 x 14k) across the bus -> tau = 28.0 s, 56.4 s to 60 V; 3.6 W at 450 V (was 74.8k -> 75.4 s, FAILED - D025) Active discharge: < 60 V within 5 s, commanded | 880R + SiC FET -> tau 0.44 s, 0.89 s to 60 V; 230 W single-shot HARDWARE-INHIBITED while CONTACTOR_EN is asserted (U402)"
- note removed: "Active discharge (SPEC 7.2): R421-R424, 4x 220R = 880R, in series with Q403 (C3M0350120J, 1200 V SiC). ~0.51 A initial at 450 V, ~230 W initial pulse for <5 s - single-shot thermal rating [TBV], not continuous. Series string per SPEC 8.2 - no single resistor spans 450 V."
- note removed: "K401: coil is in the LV 12 V domain, contacts switch the HV DC bus - the relay itself is the isolation barrier and must be rated for it: HV DC precharge relay, >=450 V DC contact rating [TBV] (e.g. TE KILOVAC or Panasonic AEV class)."
- note removed: "Passive bleeder: series string, >=4 resistors per SPEC 8.2 - no single part may span 450 V. 4x 18.7k = 74.8k -> tau = 30 s (SPEC 7.2); 2.7 W total at 450 V, ~0.68 W per part -> 3 W parts [TBV]."
- note removed: "R401: E = 0.5*C*V^2 = 40.5 J (400 uF, 450 V) -> >=41 J, >=50 W pulse [TBV]. (D013: 750 uF Si path -> 76 J; SiC chosen (D016), 400 uF stands.)"
- note removed: "SPEC 7.2 discharge requirements: Passive bleeder: < 60 V within 60 s | 75k across bus -> tau = 30 s; 2.7 W at 450 V Active discharge: < 60 V within 5 s, commanded | switched resistor, thermally rated for single-shot"
- note removed: "VOM1271 photovoltaic drive — no supply needed; ~10 s-class turn-on at µA charge currents is acceptable for discharge duty; Rds elevated at ~8 V VGS (not spec'd below 11 V) — verified acceptable for current-limited single-shot duty (D022 research)."
- moved on the sheet: D401
