File: mcuc_inverter/aux_power.kicad_sch (KiCad schematic)
At the start: 136 parts, among them Q601 CSD18543Q3A-class [TBV], Q602 CSD18543Q3A-class [TBV], Q603 CSD18543Q3A-class [TBV], Q604 CSD18543Q3A-class [TBV], Q605 CSD18543Q3A-class [TBV], T601 custom flyback per DER-948Q T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, T602 750316856, T603 750316856, T604 750316856, T605 750316856, U601 INN3990CQ, U603 LM5175RHFR, U604 LM74610QDGKRQ1, U605 LMR33630ADDAR, U606 LMR33630ADDAR, U607 TLV1117-33, U608 NXE2S0505MC, U609 SN6505BDBVR, U610 SN6505BDBVR, U611 SN6505BDBVR, U612 SN6505BDBVR

Commit message: Aux power: gate-rail post-regulation, input protection, TVS corrected
The gate-supply rails are now genuinely inside the module's absolute
maximum. The zener swap alone was not enough: the raw secondary
reaches ~24.9 V peak-charged at light load, putting V_GS(on) at
20.3 V against a +19 V AMR. Each of the four isolated domains now has
a 15 V reference plus an emitter follower, giving V_GS(on)
14.2-16.2 V over 0-70 C - 2.8 V under the limit. V_GS(off) lands at
4.84 V against the -5 V static maximum.

Two things the agent found that my instructions had wrong:
- The low-side domain draws 110 mA, not the 41 mA I quoted, because
  VGD_LS_P feeds three drivers rather than one. Its pass device
  dissipates 0.48 W and needs >=600 mm2 of tab copper - noted on the
  sheet so layout cannot miss it.
- Every BZX384-B4V7 and B15 variant is at zero stock with a 30-week
  lead, so the parts I specified were unbuyable; stocked equivalents
  substituted.

MN-14: aux input protection fitted - bidirectional TVS, P-FET reverse
polarity with the mandatory gate clamp (the full input appears
gate-to-source in this topology, so an unclamped gate dies at 24 V),
and an on-sheet note that this is explicitly NOT a load-dump design.

TVS changed SMCJ40CA -> SMCJ36CA. The 40 V part clamps at 64.5 V,
above both the LM5175's 60 V absolute maximum and the P-FET's 60 V
VDSS - it would have destroyed the devices it exists to protect. The
36 V part clamps at 58.1 V, inside both. Its standoff sits at a 24 V
jump start where leakage is microamp-class for the 60 s, which is the
right trade.

Residual documented on-sheet: the off-rail zener tempco reaches
5.06 V at -40 C and SPEC 11.5 sets no cold minimum, so -40 C
operation would need a 4.3 V part.

ERC 0 errors.

Co-Authored-By: Claude Fable 5 <noreply@anthropic.com>
Parts:
- added C684, C685, C686, C687: 10uF 25V X7R, Capacitor_SMD:C_0805_2012Metric, symbol Device:C
- added D621, D622, D623, D624: MMSZ5245C-E3-08 15V 2%, Diode_SMD:D_SOD-123, symbol Device:D_Zener
- added D625, D626, D627, D628: 1N4148W-7-F, Diode_SMD:D_SOD-123, symbol Device:D
- added D629: SMCJ36CA, Diode_SMD:D_SMC, symbol Device:D_TVS
- added D630: MMSZ5243BT1G 13V, Diode_SMD:D_SOD-123, symbol Device:D_Zener
- added Q606, Q607, Q608, Q609: BCP56-16T1G, Package_TO_SOT_SMD:SOT-223-3_TabPin2, symbol Transistor_BJT:Q_NPN_BCE
- added Q610: DMP6023LE-13, Package_TO_SOT_SMD:SOT-223-3_TabPin2, symbol Transistor_FET:Q_PMOS_GDS
- added R644, R645, R646, R647: 470R 1%, Resistor_SMD:R_0603_1608Metric, symbol Device:R
- added R648: 100k, Resistor_SMD:R_0603_1608Metric, symbol Device:R
- D607, D610, D613, D616: value BZX384-C5V1 [TBV] -> MM3Z4V7ST1G 4.7V
Connections:
- net AUX_IN: now also D629.1 (A1), Q610.2 (D); no longer C620.1, C621.1, Q601.5 (D), R620.1, U603.27 (VIN), U603.28 (VISNS)
- net GND: now also D629.2 (A2), R648.2
- net VGD_HS1_COM: now also C684.2, D621.2 (A)
- net VGD_HS1_P: now also C684.1, Q606.3 (E); no longer C662.1, C663.1, D605.1 (K), D606.1 (K)
- net VGD_HS2_COM: now also C685.2, D622.2 (A)
- net VGD_HS2_P: now also C685.1, Q607.3 (E); no longer C668.1, C669.1, D608.1 (K), D609.1 (K)
- net VGD_HS3_COM: now also C686.2, D623.2 (A)
- net VGD_HS3_P: now also C686.1, Q608.3 (E); no longer C674.1, C675.1, D611.1 (K), D612.1 (K)
- net VGD_LS_COM: now also C687.2, D624.2 (A)
- net VGD_LS_P: now also C687.1, Q609.3 (E); no longer C680.1, C681.1, D614.1 (K), D615.1 (K)
- new net: D623.1 (K), D627.1 (K)
- new net: D627.2 (A), Q608.1 (B), R646.2
- new net: D626.2 (A), Q607.1 (B), R645.2
- new net: D628.2 (A), Q609.1 (B), R647.2
- new net: D624.1 (K), D628.1 (K)
- new net: D630.2 (A), Q610.1 (G), R648.1
- new net: D622.1 (K), D626.1 (K)
- new net: D621.1 (K), D625.1 (K)
- new net: D625.2 (A), Q606.1 (B), R644.2
- new net AUX_IN_P: C620.1, C621.1, D630.1 (K), Q601.5 (D), Q610.3 (S), R620.1, U603.27 (VIN), U603.28 (VISNS)
- new net VGD_HS1_RAW: C662.1, C663.1, D605.1 (K), D606.1 (K), Q606.2 (C), R644.1
- new net VGD_HS2_RAW: C668.1, C669.1, D608.1 (K), D609.1 (K), Q607.2 (C), R645.1
- new net VGD_HS3_RAW: C674.1, C675.1, D611.1 (K), D612.1 (K), Q608.2 (C), R646.1
- new net VGD_LS_RAW: C680.1, C681.1, D614.1 (K), D615.1 (K), Q609.2 (C), R647.1
Other:
- note added: "COM-4.7 V"
- note added: "D026 - +15 V GATE RAIL POST-REGULATION. REQUIRED: the raw rail alone breaks the module AMR. Raw secondary = 5 V +-2.5% x 4.67 = 22.77-23.93 V per half, less the SS310 Vf; at light load the leakage peak-charges the reservoir to ~24.9 V. Minus the COM zener that is V_GS(on) = 20.3 V against the FS02MR12A8MA2B +19 V ABSOLUTE MAXIMUM - a continuous overstress on all six switches. A zener swap alone d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"
- note added: "Gate-drive supplies (x4): SN6505B push-pull from +5V (SN6505B is 5 V-only, D020) + WE 750316856 (1:4.67 CT:CT) -> 22-25 V raw full-wave rail (VGD_x_RAW). MM3Z4V7ST1G zener from raw(-) sets COM 4.7 V above it, so COM-N = -4.7 V; the +15 V leg is then POST-REGULATED per D026 (see the note at the left of this sheet) because the raw 20.3 V broke the module's +19 V AMR. Transformer isolation is functi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"
- note added: "HS1 +15 V post-regulator (D026)"
- note added: "HS2 +15 V post-regulator (D026)"
- note added: "HS3 +15 V post-regulator (D026)"
- note added: "LS +15 V post-regulator (D026)"
- note added: "MN-14 FIXED - AUX INPUT PROTECTION (12-24 V feed, J1203 on the comms sheet). Previously a reversed connection ran straight through the LM5175 body diodes with nothing in the way. D629 SMCJ36CA - BIDIRECTIONAL TVS, DO-214AB. Littelfuse SMCJ datasheet: V_RWM 36 V, V_C 58.1 V at rated I_PP at I_T 1 mA, 1500 W bidirectional. 36 V standoff is chosen so a 24 V system's 36 V / 60 s jump start does NOT d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"
- note added: "RAW"
- note removed: "+17.9 V"
- note removed: "-5.1 V"
- note removed: "Gate-drive supplies (x4): SN6505B push-pull from +5V (SN6505B is 5 V-only, D020) + WE 750316856 (1:4.67 CT:CT) -> ~23 V raw full-wave rail. BZX384-C5V1 zener from raw(-) sets COM 5.1 V above it: P-COM = +17.9 V, COM-N = -5.1 V. Transformer isolation is functional (2.5 kVac); the reinforced barrier remains in the 1ED3491 drivers (SPEC 5, D017). Net names match gate_drive sheet pins."
