File: mcuc_inverter/mcuc_inverter.kicad_pcb (KiCad board)
At the start: 4 copper layers, 200 x 132 mm, 564 parts, among them J1101 Coldplate NTC, J1201 CAN bus (H/L/GND/nc), J1202 GCT USB4085-GF-A, J1203 Aux 12-24 V in, J1204 Main contactor coil, J1205 Hall + motor temp, J1206 Encoder / SinCos, J1207 Resolver, J1208 FTSH-105-01-L-DV-K, J401 DC_INPUT_P tap - 6.3mm FASTON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, J402 to R401 chassis - 6.3mm FASTO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, J403 R401 return to DC_BUS_P tap -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, J404 from R424 chassis - 6.3mm FAS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, J405 DC_BUS_N tap - 6.3mm FASTON /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, J406 PHASE_U motor output stud - M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, J407 PHASE_V motor output stud - M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, J408 PHASE_W motor output stud - M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, J501 HOYS U harness - JST PA B05B-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, J502 HOYS V harness - JST PA B05B-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, J503 HOYS W harness - JST PA B05B-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, K401 HFE80V-20C/450-12-HTPAJ, Q311 BSS316N, Q321 BSS316N, Q331 BSS316N, Q341 BSS316N, Q351 BSS316N, Q361 BSS316N, Q401 NVR5198NLT1G, Q402 DMN6068LK3-13, Q403 C3M0350120J [TBV], Q404 BSS138, Q601 CSD18543Q3A-class [TBV], Q602 CSD18543Q3A-class [TBV], Q603 CSD18543Q3A-class [TBV], Q604 CSD18543Q3A-class [TBV], Q605 CSD18543Q3A-class [TBV], Q606 BCP56-16T1G, Q607 BCP56-16T1G, Q608 BCP56-16T1G, Q609 BCP56-16T1G, Q610 DMP6023LE-13, T601 custom flyback per DER-948Q T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, T602 750316856, T603 750316856, T604 750316856, T605 750316856, T701 750313734, U1 STM32F405VGT6, U1201 ISO1042DWR, U1202 USBLC6-2SC6, U201 FS02MR12A8MA2B, U301 1ED3491MC12M, U302 1ED3491MC12M, U303 1ED3491MC12M, U304 1ED3491MC12M, U305 1ED3491MC12M, U306 1ED3491MC12M, U401 VOM1271T, U402 SN74LVC1G97DBVR, U504 TLV7022DDFR, U505 TLV7022DDFR, U506 TLV7022DDFR, U507 OPA376AIDBVR, U508 OPA376AIDBVR, U509 OPA376AIDBVR, U601 INN3990CQ, U603 LM5175RHFR, U604 LM74610QDGKRQ1, U605 LMR33630ADDAR, U606 LMR33630ADDAR, U607 TLV1117-33, U608 NXE2S0505MC, U609 SN6505BDBVR, U610 SN6505BDBVR, U611 SN6505BDBVR, U612 SN6505BDBVR, U701 AMC1311BDWV, U702 MCP1804T-3302I/OT, U703 TLV9061/OPA320-class [TBV], U704 SN6505BDBVR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

Commit message: Complete collision-checked PCB routing and zone refill pass; 0 DRC clearance errors
Routing:
- net Net-(J1202-D--PadA7): track 44.6 -> 21.9 mm
- net /Communications/VBUS_DET: track 52.7 -> 32.9 mm, vias 3 -> 2
- net /Auxiliary power/FB_5V: track 44.1 -> 26.9 mm
- net /Auxiliary power/DC_BUS_P: track 0.00 -> 12.1 mm
- net Net-(R612-Pad2): track 0.00 -> 9.53 mm
- net /Phase current sensing/HOYS_V_REF: track 49.9 -> 40.8 mm
- net /Auxiliary power/BB_FB: track 23.3 -> 15.1 mm
- net /Precharge and contactor/Q403_G: track 0.00 -> 7.15 mm
- net Net-(R603-Pad2): track 0.00 -> 5.56 mm
- net /Bus voltage sensing/5V5_HV_RAW: track 0.00 -> 4.84 mm
- net /Auxiliary power/VGD_HS3_RAW: track 72.1 -> 67.4 mm
- net Net-(U801-B): track 31.2 -> 26.4 mm
- net /VGD_HS3_COM: track 63.8 -> 59.5 mm
- net /Communications/HALL_1_IN: track 27.5 -> 23.4 mm
- net /Precharge and contactor/DC_BUS_N: track 15.2 -> 12.0 mm
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