File: mcuc_inverter/mcuc_inverter.kicad_pcb (KiCad board)
At the start: 4 copper layers, 200 x 132 mm, 564 parts, among them J1101 Coldplate NTC, J1201 CAN bus (H/L/GND/nc), J1202 GCT USB4085-GF-A, J1203 Aux 12-24 V in, J1204 Main contactor coil, J1205 Hall + motor temp, J1206 Encoder / SinCos, J1207 Resolver, J1208 FTSH-105-01-L-DV-K, J401 DC_INPUT_P tap - 6.3mm FASTON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, J402 to R401 chassis - 6.3mm FASTO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, J403 R401 return to DC_BUS_P tap -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, J404 from R424 chassis - 6.3mm FAS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, J405 DC_BUS_N tap - 6.3mm FASTON /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, J406 PHASE_U motor output stud - M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, J407 PHASE_V motor output stud - M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, J408 PHASE_W motor output stud - M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, J501 HOYS U harness - JST PA B05B-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, J502 HOYS V harness - JST PA B05B-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, J503 HOYS W harness - JST PA B05B-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, K401 HFE80V-20C/450-12-HTPAJ, Q311 BSS316N, Q321 BSS316N, Q331 BSS316N, Q341 BSS316N, Q351 BSS316N, Q361 BSS316N, Q401 NVR5198NLT1G, Q402 DMN6068LK3-13, Q403 C3M0350120J [TBV], Q404 BSS138, Q601 CSD18543Q3A-class [TBV], Q602 CSD18543Q3A-class [TBV], Q603 CSD18543Q3A-class [TBV], Q604 CSD18543Q3A-class [TBV], Q605 CSD18543Q3A-class [TBV], Q606 BCP56-16T1G, Q607 BCP56-16T1G, Q608 BCP56-16T1G, Q609 BCP56-16T1G, Q610 DMP6023LE-13, T601 custom flyback per DER-948Q T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, T602 750316856, T603 750316856, T604 750316856, T605 750316856, T701 750313734, U1 STM32F405VGT6, U1201 ISO1042DWR, U1202 USBLC6-2SC6, U201 FS02MR12A8MA2B, U301 1ED3491MC12M, U302 1ED3491MC12M, U303 1ED3491MC12M, U304 1ED3491MC12M, U305 1ED3491MC12M, U306 1ED3491MC12M, U401 VOM1271T, U402 SN74LVC1G97DBVR, U504 TLV7022DDFR, U505 TLV7022DDFR, U506 TLV7022DDFR, U507 OPA376AIDBVR, U508 OPA376AIDBVR, U509 OPA376AIDBVR, U601 INN3990CQ, U603 LM5175RHFR, U604 LM74610QDGKRQ1, U605 LMR33630ADDAR, U606 LMR33630ADDAR, U607 TLV1117-33, U608 NXE2S0505MC, U609 SN6505BDBVR, U610 SN6505BDBVR, U611 SN6505BDBVR, U612 SN6505BDBVR, U701 AMC1311BDWV, U702 MCP1804T-3302I/OT, U703 TLV9061/OPA320-class [TBV], U704 SN6505BDBVR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

Commit message: Phase B routing continued: 421 -> 203 unconnected; commit the router tooling
Collision-checked completion routing on the control board: 218 open
connections closed, 0 error-severity DRC violations throughout (kicad-cli
9.0.6, zones refilled before every check). Board now carries 6052 track
segments and 1188 vias.

The remaining 203 opens are the congested residue (fine-pitch PWM gating
blocks, HV-relax pockets) where legal lanes are exactly minimum-clearance
wide; they need a push-and-shove router. The tooling that did the rest is
committed under tools/pcb_router/ -- the 2026-08-04 session's router never
entered version control, and that practice ends here.

Also removed 25 stacked same-net vias (holes_co_located 85 -> 0,
hole_to_hole 4 -> 0). Full account in docs/CHANGELOG.md.

Co-Authored-By: Claude Fable 5 <noreply@anthropic.com>
Routing:
- net GND: track 573.5 -> 848.7 mm, vias 210 -> 257
- net +5V: track 337.2 -> 506.2 mm, vias 36 -> 60
- net /Auxiliary power/DC_BUS_P: track 12.1 -> 175.9 mm, vias 0 -> 2
- net +3.3V: track 829.8 -> 987.3 mm, vias 104 -> 130
- net Net-(D401-A): track 22.6 -> 134.9 mm, vias 0 -> 3
- net Net-(U802B-+): track 2.61 -> 104.1 mm, vias 0 -> 7
- net +12V: track 164.3 -> 261.8 mm, vias 4 -> 17
- net Net-(D605-A): track 0.00 -> 91.2 mm, vias 0 -> 6
- net Net-(D615-A): track 0.00 -> 88.2 mm, vias 0 -> 4
- net /Phase current sensing/OC_TRIP: track 63.2 -> 139.6 mm, vias 3 -> 9
- net Net-(U801-CLKIN): track 0.00 -> 73.9 mm, vias 0 -> 2
- net /Auxiliary power/BB_COMP: track 0.00 -> 73.4 mm, vias 0 -> 4
- net /HALL_3: track 0.00 -> 71.9 mm, vias 0 -> 2
- net Net-(R616-Pad2): track 0.00 -> 70.9 mm, vias 0 -> 2
- net /Auxiliary power/AUX_15V: track 89.9 -> 160.3 mm, vias 9 -> 15
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